File: pcb/airsmiley.kicad_pcb (KiCad board)
At the start: 2 copper layers, 56 x 49 mm, 12 parts, among them J1 Conn_01x02, U1 WeMos_D1_mini

Commit message: Renamed to "Air Smiley"
Parts:
- added J_RST_1: Conn_01x02, Connector_PinHeader_2.54mm:PinHeader_1x02_P2.54mm_Vertical, F.Cu at (129.5, 78.7)
- moved J_WS2812B_1 5.08 mm to (124.5, 76.2)
Connections:
- U1 pad 12: (no net) -> Net-(U1-Pad12)
- U1 pad 16: (no net) -> Net-(U1-Pad16)
- U1 pad 2: (no net) -> Net-(U1-Pad2)
- U1 pad 4: (no net) -> Net-(U1-Pad4)
- U1 pad 5: (no net) -> Net-(U1-Pad5)
- U1 pad 6: (no net) -> Net-(U1-Pad6)
- U1 pad 7: (no net) -> Net-(U1-Pad7)
Routing:
- net GND: track 126.3 -> 141.1 mm
- net Net-(J1-Pad1): track 6.13 -> 12.3 mm
- net TO_DI: track 20.8 -> 24.4 mm
- net +5V: track 68.2 -> 69.4 mm
Other:
- board text added: "Air Smiley 2021 HTL Weiz v1"
- board text added: "RST"
- board text removed: "CO2box 2020 HTL Weiz"

Commit message: minor pcb changes
Parts:
- added Ref**: Val**, airsmiley:logo, B.Cu at (146.0, 104.7)
- added Ref**: Val**, airsmiley:logo, F.Cu at (154.0, 105.7)
Other:
- board text added: "Air Smiley 2021 v1"
- board text removed: "Air Smiley 2021 HTL Weiz v1"
